File: pcb/Control-Panel/Control-Panel.kicad_pcb (KiCad board)
At the start: 2 copper layers, 211 x 40.2 mm, 0 parts

Commit message: Critical mechanical parts placement.
Parts:
- added C1: 100nF, Capacitor_SMD:C_0603_1608Metric, B.Cu at (80.1, 98.0)
- added C2: 4.7uF, Capacitor_SMD:C_0603_1608Metric, B.Cu at (81.4, 92.8)
- added C3: 4.7uF, Capacitor_SMD:C_0603_1608Metric, B.Cu at (74.8, 87.3)
- added C4: 1uF, Capacitor_SMD:C_0603_1608Metric, B.Cu at (81.4, 95.3)
- added C5: 1uF, Capacitor_SMD:C_0603_1608Metric, B.Cu at (74.8, 89.8)
- added C6: 100nF, Capacitor_SMD:C_0603_1608Metric, B.Cu at (70.5, 83.8)
- added C7: 4.7uF, Capacitor_SMD:C_0603_1608Metric, B.Cu at (84.1, 97.8)
- added C8: 10uF, Capacitor_Tantalum_SMD:CP_EIA-3216-18_Kemet-A, B.Cu at (69.1, 97.0)
- added D1: MBR0520L, Diode_SMD:D_SOD-123, B.Cu at (81.0, 100.9)
- added DS1: UG-2864KSWLG01, Display:OLED-128O064D, F.Cu at (77.0, 91.2)
- added F1: 350mA, Fuse:Fuse_0603_1608Metric_Castellated, B.Cu at (68.5, 94.2)
- added J1: Conn_01x08, Connector_JST:JST_PH_S8B-PH-SM4-TB_1x08-1MP_P2.00mm_Horizontal, F.Cu at (109.0, 84.0)
- added JP1: A0, Jumper:SolderJumper-2_P1.3mm_Bridged_RoundedPad1.0x1.5mm, B.Cu at (72.8, 92.8)
- added JP2: A1, Jumper:SolderJumper-2_P1.3mm_Bridged_RoundedPad1.0x1.5mm, B.Cu at (86.0, 100.8)
- added JP3: A2, Jumper:SolderJumper-2_P1.3mm_Bridged_RoundedPad1.0x1.5mm, B.Cu at (77.2, 92.8)
- added JP4: SA0, Jumper:SolderJumper-2_P1.3mm_Open_RoundedPad1.0x1.5mm, B.Cu at (70.7, 89.3)
- added R1: 10k, Resistor_SMD:R_0603_1608Metric, B.Cu at (70.5, 86.3)
- added R2: 10k, Resistor_SMD:R_0603_1608Metric, B.Cu at (88.1, 97.8)
- added R3: 10k, Resistor_SMD:R_0603_1608Metric, B.Cu at (74.5, 82.3)
- added R4: 4.7k, Resistor_SMD:R_0603_1608Metric, B.Cu at (85.4, 92.8)
- added R5: 10k, Resistor_SMD:R_0603_1608Metric, B.Cu at (78.8, 87.3)
- added R6: 10k, Resistor_SMD:R_0603_1608Metric, B.Cu at (78.8, 89.8)
- added R7: 560k, Resistor_SMD:R_0603_1608Metric, B.Cu at (85.4, 95.3)
- added R8: 10k, Resistor_SMD:R_0603_1608Metric, B.Cu at (74.5, 84.8)
- added SW1: SW_Push, private:MembraneButton_GrandPianist, F.Cu at (124.6, 92.3)
- added SW10: SW_Push, private:MembraneButton_GrandPianist, F.Cu at (238.9, 95.8)
- added SW2: SW_Push, private:MembraneButton_GrandPianist, F.Cu at (141.9, 92.3)
- added SW3: SW_Push, private:MembraneButton_GrandPianist, F.Cu at (159.1, 92.3)
- added SW4: SW_Push, private:MembraneButton_GrandPianist, F.Cu at (175.9, 91.1)
- added SW5: SW_Push, private:MembraneButton_GrandPianist, F.Cu at (188.6, 86.6)
- added SW6: SW_Push, private:MembraneButton_GrandPianist, F.Cu at (188.6, 95.8)
- added SW7: SW_Push, private:MembraneButton_GrandPianist, F.Cu at (201.3, 91.1)
- added SW8: SW_Push, private:MembraneButton_GrandPianist, F.Cu at (218.1, 91.7)
- added SW9: SW_Push, private:MembraneButton_GrandPianist, F.Cu at (238.9, 86.6)
- added U1: MCP23017_SS, Package_SO:SSOP-28_5.3x10.2mm_P0.65mm, B.Cu at (112.8, 91.8)
Routing:
- added copper zone on B.Cu, net (none)
- added copper zone on F.Cu, net (none)
Other:
- board text added: "Grand Pianist++ Control Panel v0.0.0"
