File: pcb/Control-Panel/Control-Panel.sch (KiCad schematic (older format))
At the start: 35 parts, among them J1 Conn_01x08, SW1 SW_Push, SW10 SW_Push, SW2 SW_Push, SW3 SW_Push, SW4 SW_Push, SW5 SW_Push, SW6 SW_Push, SW7 SW_Push, SW8 SW_Push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

Commit message: Critical mechanical parts placement.
Parts:
- DS1: value OLED-128O064D -> UG-2864KSWLG01; Field4 (none) -> https://datasheet.lcsc.com/lcsc/Univision-Semicon-UG-2864KS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
Changed lines of the file:
@@
 P 3500 4750
 F 0 "DS1" H 3100 6200 50  0000 L CNN
-F 1 "OLED-128O064D" H 3650 6200 50  0000 L CNN
+F 1 "UG-2864KSWLG01" H 3650 6200 50  0000 L CNN
 F 2 "Display:OLED-128O064D" H 3500 4750 50  0001 C CNN
 F 3 "https://www.vishay.com/docs/37902/oled128o064dbpp3n00000.pdf" H 3500 5550 50  0001 C CNN
+F 4 "https://datasheet.lcsc.com/lcsc/Univision-Semicon-UG-2864KSWMG01_C88331.pdf" H 3500 4750 50  0001 C CNN "Field4"
 	1    3500 4750
 	1    0    0    -1
